File: catalyst46_v1/catalyst.kicad_pcb (KiCad board)
At the start: 2 copper layers, 312.6 x 121.2 mm, 47 parts, among them U1 RP2040-Zero

Commit message: Added copper pour zones
Connections:
- U1 pad GND: (no net) -> gnd
Routing:
- net gnd: track 0.00 -> 6.59 mm
- added copper zone on B.Cu, net gnd
- added copper zone on F.Cu, net gnd
Changed lines of the file:
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@@
 			(layers "*.Cu" "*.Mask")
 			(remove_unused_layers no)
+			(net "gnd")
 		)
 		(embedded_fonts no)
@@
 		(net "C7")
 	)
+	(segment
+		(start 216.112158 62.862158)
+		(end 217.38 64.13)
+		(width 0.25)
+		(layer "F.Cu")
+		(net "gnd")
+	)
+	(segment
+		(start 217.38 64.13)
+		(end 215 64.13)
+		(width 0.25)
+		(layer "F.Cu")
+		(net "gnd")
+	)
+	(segment
+		(start 216.107532 65.402468)
+		(end 215.8 65.402468)
+		(width 0.25)
+		(layer "F.Cu")
+		(net "gnd")
+	)
+	(segment
+		(start 215.8 62.862158)
+		(end 216.112158 62.862158)
+		(width 0.25)
+		(layer "F.Cu")
+		(net "gnd")
+	)
+	(segment
+		(start 217.38 64.13)
+		(end 216.107532 65.402468)
+		(width 0.25)
+		(layer "F.Cu")
+		(net "gnd")
+	)
+	(zone
+		(net "gnd")
+		(layers "F.Cu" "B.Cu")
+		(hatch edge 0.5)
+		(connect_pads
+			(clearance 0.6)
+		)
+		(min_thickness 0.25)
+		(fill yes
+			(thermal_gap 0.5)
+			(thermal_bridge_width 0.5)
+			(smoothing fillet)
+			(radius 3)
+			(island_removal_mode 0)
+		)
+		(polygon
+			(pts
+				(xy 64.6 28.2) (xy 389.4 28.2) (xy 389.4 172.2) (xy 64.6 172.2)
+			)
+		)
+	)
 	(embedded_fonts no)
